Commit message: Task - 1

File: my_rb1_description/urdf/my_rb1_robot.urdf (robot description, URDF)
Before this commit: robot robot, 6 links, 5 joints
Links:
- added link base_footprint
Joints:
- added joint base_joint: type fixed, parent base_footprint, child base_link, origin xyz=0 0 0.0102 rpy=0 0 0

Commit message: First RB1 commit

File: my_rb1_description/urdf/my_rb1_robot.urdf (robot description, URDF)
Before this commit: robot robot, 7 links, 6 joints
Links:
- link base_footprint: geometry collision box size=0.2 0.1 0.01
- link front_caster: geometry collision sphere radius=0.015; collision sphere radius=0.025
Joints:
- joint base_joint: child base_link -> base_footprint; origin xyz=0 0 0.0102 rpy=0 0 0 -> xyz=0 0 -0.15 rpy=0 0 0; parent base_footprint -> base_link
- joint joint_back_caster: origin xyz=0.1 0 -0.15 rpy=0 0 0 -> xyz=-0.1 0 -0.15 rpy=0 0 0
- joint joint_front_caster: origin xyz=-0.1 0 -0.15 rpy=0 0 0 -> xyz=0.1 0 -0.15 rpy=0 0 0
